File: USB_C_Daughterboard/USB_C_Daughterboard.kicad_pcb (KiCad board)
At the start: 2 copper layers, 10.8 x 14 mm, 11 parts, among them J1 USB_C_Receptacle_USB2.0

Commit message: Rename daughterboard nets for better PCBnew labeling
Connections:
- net Net-(H1-Pad1) renamed /D-
- net Net-(H2-Pad1) renamed /D+
- net Net-(H3-Pad1) renamed /SBU1
- net Net-(H4-Pad1) renamed /SBU2
- net Net-(J1-PadA5) renamed /CC1
- net Net-(J1-PadB5) renamed /CC2
